File: AEDR-7810-Breakout.brd (EAGLE design)
At the start: 15.2 x 12.7 mm, 8 parts, among them J1 1X5, U1 AEDR-871X

Commit message: Completed initial rev of breakout
Parts:
- removed J1: 1X5, headers.edge(.1in):1X5
- added H1: 2X5, headers(.1in):2X5
- added H2: 1X5, headers(.1in):1X5
- J2, J3: device solderjumper:3.LRG.12 -> solderjumper:3.MED.12
- moved C2 11.5 mm to (2.86, 2.22), turned to 180 degrees
- moved J2 11.3 mm to (1.91, 5.08)
- moved C1 10.9 mm to (12.4, 2.22), turned to 0 degrees
- moved J3 10.6 mm to (13.3, 5.08)
- moved C4 10.3 mm to (1.91, 3.81), turned to 180 degrees
- moved C3 9.67 mm to (13.3, 3.81), turned to 0 degrees
- moved U1 3.18 mm to (7.62, 3.81), turned to 180 degrees
Connections:
- net 3.3V: now also H1.1, H1.2; no longer J1.1
- net CHA: now also H1.7, H1.8; no longer J1.2
- net CHB: now also H1.5, H1.6; no longer J1.3
- net CHI: now also H1.3, H1.4; no longer J1.4
- net GND: now also H1.10, H1.9; no longer J1.5
Routing:
- net 3.3V: track 0.00 -> 32.0 mm, vias 0 -> 2
- net N$5: track 0.00 -> 12.9 mm, vias 0 -> 2
- net CHA: track 0.00 -> 8.24 mm
- net CHI: track 0.00 -> 7.22 mm
- net CHB: track 0.00 -> 6.78 mm
- net N$4: track 0.00 -> 6.21 mm, vias 0 -> 2
Other:
- board size 15.2 x 12.7 mm -> 15.2 x 10.8 mm
- board text added: "3.3v"
- board text added: "A"
- board text added: "AEDR-871X Breakout"
- board text added: "B"
- board text added: "Cruz Monrreal II"
- board text added: "GND"
- board text added: "I"
- board text added: "S1"
- board text added: "S2"
- board text added: "TheNextPlateau.com"
